Commit message: 4.29_12:30_update

File: src/my_simulation/models_and_worlds/simple_car.urdf (robot description, URDF)
Before this commit: robot simple_car, 8 links, 7 joints
Links:
- added link left_front_guard, mass 0.12; collision box size=0.55 0.018 0.03; visual box size=0.55 0.018 0.03
- added link left_guard_tip, mass 0.10; collision cylinder length=0.05 radius=0.04; visual cylinder length=0.05 radius=0.04
- added link right_front_guard, mass 0.12; collision box size=0.55 0.018 0.03; visual box size=0.55 0.018 0.03
- added link right_guard_tip, mass 0.10; collision cylinder length=0.05 radius=0.04; visual cylinder length=0.05 radius=0.04
Joints:
- added joint base_to_left_front_guard: type fixed, parent base_link, child left_front_guard, origin xyz=0.40 0.24 -0.005 rpy=0 0 0.60
- added joint base_to_right_front_guard: type fixed, parent base_link, child right_front_guard, origin xyz=0.40 -0.24 -0.005 rpy=0 0 -0.60
- added joint left_front_guard_to_tip: type fixed, parent left_front_guard, child left_guard_tip, origin xyz=0.305 0 0 rpy=0 0 0
- added joint right_front_guard_to_tip: type fixed, parent right_front_guard, child right_guard_tip, origin xyz=0.305 0 0 rpy=0 0 0

Commit message: 5.5_14:30_update

File: src/my_simulation/models_and_worlds/simple_car.urdf (robot description, URDF)
Before this commit: robot simple_car, 12 links, 11 joints
Links:
- link base_link: geometry collision box size=0.5 0.5 0.07; visual box size=0.5 0.5 0.07
Joints:
- joint base_to_camera: origin xyz=0.25 0 0.05 rpy=0 0 0 -> xyz=0.25 0 0.055 rpy=0 0 0
